File: robot arm/schematic.sch (EAGLE design)
At the start: 7 parts

Commit message: xixixi
Parts:
- removed DIS1: EA_DIP, display-lcd:EA_DIP
- added LIMIT_SWICH1, LIMIT_SWICH2, LIMIT_SWICH3, LIMIT_SWICH4: (no value), switch:255SB
- PCB1: value ARDUINO_UNO -> ARDUINO_UNO_EXT; device arduino:ARDUINO_UNO -> arduino:ARDUINO_UNO_EXT
- U$1: value LCD-I2C-CONVERTER -> RELAY-1-SRD; device diy-modules:LCD-I2C-CONVERTER -> diy-modules:RELAY-1-SRD
Connections:
- removed net GND: PCB1.GND.
- removed net N$18: DIS1.NC@1, U$1.LED.A
- removed net N$19: DIS1.NC@2, U$1.LED.K
- removed net N$20: DIS1.VEE, U$1.VEE
- removed net VCC: PCB1.5V
- new net +12V: STEPDRV1.VMOT, STEPDRV2.VMOT, STEPDRV3.VMOT, STEPDRV4.VMOT
- new net +5V: PCB1.VIN, STEPDRV1.MS1, STEPDRV1.MS3, STEPDRV1.VDD, STEPDRV2.MS1, STEPDRV2.MS3, STEPDRV2.VDD, STEPDRV3.MS1, STEPDRV3.MS3, STEPDRV3.VDD, STEPDRV4.MS1, STEPDRV4.MS3, STEPDRV4.VDD, U$1.VCC.1
- new net 10: LIMIT_SWICH2.O, PCB1.~10
- new net 11: LIMIT_SWICH1.O, PCB1.~11
- new net 12: PCB1.12, STEPDRV2.STEP
- new net 13: PCB1.13, STEPDRV2.DIR
- new net 2: PCB1.2, STEPDRV3.STEP
- new net 3: PCB1.~3, STEPDRV4.STEP
- new net 4: PCB1.4, STEPDRV1.STEP
- new net 5: PCB1.~5, STEPDRV3.DIR
- new net 6: PCB1.~6, STEPDRV4.DIR
- new net 7: PCB1.7, STEPDRV1.DIR
- new net 9: LIMIT_SWICH3.O, PCB1.~9
- new net A0: PCB1.A0, U$1.IN1
- new net A3: LIMIT_SWICH4.O, PCB1.A3
- new net N$3: STEPDRV1.2A
- new net N$4: STEPDRV1.1A
- new net PE: LIMIT_SWICH1.P, LIMIT_SWICH2.P, LIMIT_SWICH3.P, LIMIT_SWICH4.P, PCB1.GND., PCB1.GND.., STEPDRV1.!ENABLE, STEPDRV1.!RESET, STEPDRV1.!SLEEP, STEPDRV1.GND@0, STEPDRV1.GND@1, STEPDRV1.MS2, STEPDRV2.!ENABLE, STEPDRV2.!RESET, STEPDRV2.!SLEEP, STEPDRV2.GND@0, STEPDRV2.GND@1, STEPDRV2.MS2, STEPDRV3.!ENABLE, STEPDRV3.!RESET, STEPDRV3.!SLEEP, STEPDRV3.GND@0, STEPDRV3.GND@1, STEPDRV3.MS2, STEPDRV4.!ENABLE, STEPDRV4.!RESET, STEPDRV4.!SLEEP, STEPDRV4.GND@0, STEPDRV4.GND@1, STEPDRV4.MS2, U$1.GND
- net N$1: now also STEPDRV1.2B; no longer PCB1.A5, U$1.SCL
- net N$10: now also STEPDRV3.1B; no longer DIS1.D0, U$1.DB0
- net N$11: now also STEPDRV3.2A; no longer DIS1.D1, U$1.DB1
- net N$12: now also STEPDRV3.1A; no longer DIS1.D2, U$1.DB2
- net N$13: now also STEPDRV4.2B; no longer DIS1.D3, U$1.DB3
- net N$14: now also STEPDRV4.1B; no longer DIS1.D4, U$1.DB4
- net N$15: now also STEPDRV4.2A; no longer DIS1.D5, U$1.DB5
- net N$16: now also STEPDRV4.1A; no longer DIS1.D6, U$1.DB6
- net N$17: now also U$1.JD-VCC, U$1.VCC.2; no longer DIS1.D7, U$1.DB7
- net N$2: now also STEPDRV1.1B; no longer PCB1.A4, U$1.SDA
- net N$5: now also STEPDRV2.2B; no longer DIS1.VSS, U$1.VSS
- net N$6: now also STEPDRV2.1B; no longer DIS1.VDD, U$1.VDD
- net N$7: now also STEPDRV2.2A; no longer DIS1.RS, U$1.RS
- net N$8: now also STEPDRV2.1A; no longer DIS1.R/W, U$1.R/W
- net N$9: now also STEPDRV3.2B; no longer DIS1.E, U$1.EN
Other:
- note added: "24V"
- note added: "A"
- note added: "GND"
- note added: "JOINT 1"
- note added: "JOINT 2"
- note added: "JOINT 3"
- note added: "P"
- note added: "SOLENOID VALVE"
- note added: "Z AXIS"
- note removed: "M3"
- note removed: "M4"
- moved on the sheet: STEPDRV1, STEPDRV2, STEPDRV3, STEPDRV4
