File: Pyranometer/main board.brd (EAGLE design)
At the start: 160 x 100 mm, 9 parts

Commit message: backup
Parts:
- removed U$3: CURRENT-SENSOR-ACS712#IC, diy-modules:CURRENT-SENSOR-ACS712#IC
- added PHOTOVOLTAIC: B6B-EH-A, con-JST EH:B6B-EH-A
- moved U$1 5.68 mm to (-34.3, 29.2)
Connections:
- removed net N$6: SOLAR_CELL.1, U$3.P1.2
- net N$1: now also PHOTOVOLTAIC.6, SOLAR_CELL.1; no longer U$1.1, U$3.2
- net N$5: now also PHOTOVOLTAIC.5; no longer U$3.P1.1
- net PE: now also PHOTOVOLTAIC.2; no longer U$3.3
- net SCL: now also PHOTOVOLTAIC.3
- net SDA: now also PHOTOVOLTAIC.4
- net VCC: now also PHOTOVOLTAIC.1; no longer U$3.1
Changed lines of the file:
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@@
 <element name="SUPPLY" library="con-JST EH" package="B2B-EH-A" value="B2B-EH-A" x="-35.56" y="110.49"/>
 <element name="SWITCH" library="con-JST EH" package="B2B-EH-A" value="B2B-EH-A" x="-21.59" y="110.49"/>
-<element name="U$1" library="nodemcu(1)" package="NODEMCU" value="NODEMCU" x="-29.21" y="31.75"/>
+<element name="U$1" library="nodemcu(1)" package="NODEMCU" value="NODEMCU" x="-34.29" y="29.21"/>
 <element name="U$2" library="diy-modules" package="DC-DC-STEP-DOWN-LM2596" value="DC-DC-STEP-DOWN-LM2596" x="-35.56" y="74.93"/>
-<element name="U$3" library="diy-modules" package="CURRENT-SENSOR-ACS712#IC" value="CURRENT-SENSOR-ACS712#IC" x="-29.21" y="97.79"/>
+<element name="PHOTOVOLTAIC" library="con-JST EH" package="B6B-EH-A" value="B6B-EH-A" x="-68.58" y="-7.62"/>
 </elements>
 <signals>
@@
 <contactref element="U$1" pad="17"/>
 <contactref element="U$1" pad="24"/>
-<wire x1="-15.24" y1="16.51" x2="-43.18" y2="16.51" width="0" layer="19" extent="1-1"/>
-<wire x1="-15.24" y1="34.29" x2="-15.24" y2="16.51" width="0" layer="19" extent="1-1"/>
-<wire x1="-43.18" y1="46.99" x2="-43.18" y2="16.51" width="0" layer="19" extent="1-1"/>
+<wire x1="-20.32" y1="13.97" x2="-48.26" y2="13.97" width="0" layer="19" extent="1-1"/>
+<wire x1="-20.32" y1="31.75" x2="-20.32" y2="13.97" width="0" layer="19" extent="1-1"/>
+<wire x1="-48.26" y1="44.45" x2="-48.26" y2="13.97" width="0" layer="19" extent="1-1"/>
 </signal>
 <signal name="3V">
@@
 <contactref element="U$1" pad="16"/>
 <contactref element="U$1" pad="25"/>
-<wire x1="-15.24" y1="13.97" x2="-43.18" y2="24.13" width="0" layer="19" extent="1-1"/>
-<wire x1="-15.24" y1="36.83" x2="-15.24" y2="13.97" width="0" layer="19" extent="1-1"/>
-</signal>
-<signal name="N$1">
-<contactref element="U$1" pad="1"/>
-<contactref element="U$3" pad="2"/>
-<wire x1="-43.18" y1="49.53" x2="-15.24" y2="97.79" width="0" layer="19" extent="1-1"/>
+<wire x1="-20.32" y1="11.43" x2="-48.26" y2="21.59" width="0" layer="19" extent="1-1"/>
+<wire x1="-20.32" y1="34.29" x2="-20.32" y2="11.43" width="0" layer="19" extent="1-1"/>
 </signal>
 <signal name="N$2">
@@
 <signal name="VCC">
 <contactref element="U$2" pad="OUT+"/>
-<contactref element="U$3" pad="1"/>
 <contactref element="U$1" pad="15"/>
 <contactref element="RTC" pad="2"/>
 <contactref element="LCD" pad="2"/>
 <contactref element="DATALOGGER" pad="2"/>
-<wire x1="-15.748" y1="83.566" x2="-15.24" y2="100.33" width="0" layer="19" extent="1-1"/>
-<wire x1="-49.51" y1="110.49" x2="-15.24" y2="100.33" width="0" layer="19" extent="1-1"/>
+<contactref element="PHOTOVOLTAIC" pad="1"/>
+<wire x1="-48.26" y1="11.43" x2="-74.83" y2="-7.62" width="0" layer="19" extent="1-1"/>
+<wire x1="-15.748" y1="83.566" x2="-48.26" y2="11.43" width="0" layer="19" extent="1-1"/>
+<wire x1="-49.51" y1="110.49" x2="-15.748" y2="83.566" width="0" layer="19" extent="1-1"/>
 <wire x1="-64.75" y1="110.49" x2="-49.51" y2="110.49" width="0" layer="19" extent="1-1"/>
 <wire x1="-58.36" y1="93.98" x2="-64.75" y2="110.49" width="0" layer="19" extent="1-1"/>
-<wire x1="-43.18" y1="13.97" x2="-15.748" y2="83.566" width="0" layer="19" extent="1-1"/>
 </signal>
 <signal name="PE">
 <contactref element="U$2" pad="OUT-"/>
-<contactref element="U$3" pad="3"/>
 <contactref element="U$1" pad="10"/>
 <contactref element="RTC" pad="1"/>
 <contactref element="LCD" pad="1"/>
 <contactref element="DATALOGGER" pad="1"/>
-<wire x1="-15.748" y1="66.294" x2="-15.24" y2="95.25" width="0" layer="19" extent="1-1"/>
-<wire x1="-52.01" y1="110.49" x2="-15.24" y2="95.25" width="0" layer="19" extent="1-1"/>
-<wire x1="-67.25" y1="110.49" x2="-52.01" y2="110.49" width="0" layer="19" extent="1-1"/>
-<wire x1="-60.86" y1="93.98" x2="-67.25" y2="110.49" width="0" layer="19" extent="1-1"/>
-<wire x1="-43.18" y1="26.67" x2="-15.748" y2="66.294" width="0" layer="19" extent="1-1"/>
-</signal>
-<signal name="N$5">
-<contactref element="U$3" pad="P1.1"/>
-<contactref element="SOLAR_CELL" pad="2"/>
-<wire x1="-72.41" y1="92.71" x2="-40.64" y2="100.33" width="0" layer="19" extent="1-1"/>
-</signal>
-<signal name="N$6">
-<contactref element="SOLAR_CELL" pad="1"/>
-<contactref element="U$3" pad="P1.2"/>
-<wire x1="-74.91" y1="92.71" x2="-40.64" y2="95.25" width="0" layer="19" extent="1-1"/>
+<contactref element="PHOTOVOLTAIC" pad="2"/>
+<wire x1="-48.26" y1="24.13" x2="-72.33" y2="-7.62" width="0" layer="19" extent="1-1"/>
+<wire x1="-15.748" y1="66.294" x2="-48.26" y2="24.13" width="0" layer="19" extent="1-1"/>
+<wire x1="-60.86" y1="93.98" x2="-15.748" y2="66.294" width="0" layer="19" extent="1-1"/>
+<wire x1="-67.25" y1="110.49" x2="-60.86" y2="93.98" width="0" layer="19" extent="1-1"/>
+<wire x1="-52.01" y1="110.49" x2="-67.25" y2="110.49" width="0" layer="19" extent="1-1"/>
 </signal>
 <signal name="SCL">
@@
 <contactref element="RTC" pad="4"/>
 <contactref element="LCD" pad="4"/>
+<contactref element="PHOTOVOLTAIC" pad="3"/>
+<wire x1="-20.32" y1="44.45" x2="-69.83" y2="-7.62" width="0" layer="19" extent="1-1"/>
+<wire x1="-44.51" y1="110.49" x2="-20.32" y2="44.45" width="0" layer="19" extent="1-1"/>
 <wire x1="-59.75" y1="110.49" x2="-44.51" y2="110.49" width="0" layer="19" extent="1-1"/>
-<wire x1="-15.24" y1="46.99" x2="-44.51" y2="110.49" width="0" layer="19" extent="1-1"/>
 </signal>
 <signal name="SDA">
@@
 <contactref element="RTC" pad="3"/>
 <contactref element="LCD" pad="3"/>
+<contactref element="PHOTOVOLTAIC" pad="4"/>
+<wire x1="-20.32" y1="41.91" x2="-67.33" y2="-7.62" width="0" layer="19" extent="1-1"/>
+<wire x1="-47.01" y1="110.49" x2="-20.32" y2="41.91" width="0" layer="19" extent="1-1"/>
 <wire x1="-62.25" y1="110.49" x2="-47.01" y2="110.49" width="0" layer="19" extent="1-1"/>
-<wire x1="-15.24" y1="44.45" x2="-47.01" y2="110.49" width="0" layer="19" extent="1-1"/>
 </signal>
 <signal name="CS">
 <contactref element="DATALOGGER" pad="6"/>
 <contactref element="U$1" pad="7"/>
-<wire x1="-43.18" y1="34.29" x2="-48.36" y2="93.98" width="0" layer="19" extent="1-1"/>
+<wire x1="-48.26" y1="31.75" x2="-48.36" y2="93.98" width="0" layer="19" extent="1-1"/>
 </signal>
 <signal name="SCK">
 <contactref element="DATALOGGER" pad="5"/>
 <contactref element="U$1" pad="9"/>
-<wire x1="-43.18" y1="29.21" x2="-50.86" y2="93.98" width="0" layer="19" extent="1-1"/>
+<wire x1="-48.26" y1="26.67" x2="-50.86" y2="93.98" width="0" layer="19" extent="1-1"/>
 </signal>
 <signal name="MOSI">
 <contactref element="DATALOGGER" pad="4"/>
 <contactref element="U$1" pad="6"/>
-<wire x1="-43.18" y1="36.83" x2="-53.36" y2="93.98" width="0" layer="19" extent="1-1"/>
+<wire x1="-48.26" y1="34.29" x2="-53.36" y2="93.98" width="0" layer="19" extent="1-1"/>
 </signal>
 <signal name="MISO">
 <contactref element="DATALOGGER" pad="3"/>
 <contactref element="U$1" pad="8"/>
-<wire x1="-43.18" y1="31.75" x2="-55.86" y2="93.98" width="0" layer="19" extent="1-1"/>
+<wire x1="-48.26" y1="29.21" x2="-55.86" y2="93.98" width="0" layer="19" extent="1-1"/>
+</signal>
+<signal name="N$1">
+<contactref element="PHOTOVOLTAIC" pad="6"/>
+<contactref element="SOLAR_CELL" pad="1"/>
+<wire x1="-74.91" y1="92.71" x2="-62.33" y2="-7.62" width="0" layer="19" extent="1-1"/>
+</signal>
+<signal name="N$5">
+<contactref element="PHOTOVOLTAIC" pad="5"/>
+<contactref element="SOLAR_CELL" pad="2"/>
+<wire x1="-72.41" y1="92.71" x2="-64.83" y2="-7.62" width="0" layer="19" extent="1-1"/>
 </signal>
 </signals>
